Commit message: Imported upstream version '1.0.1' of 'upstream'

File: ur_description/urdf/ur5.transmission.xacro (robot description, xacro)
@@ -1,37 +1,52 @@
 <?xml version="1.0"?>
-<robot xmlns:sensor="http://playerstage.sourceforge.net/gazebo/xmlschema/#sensor"
-       xmlns:controller="http://playerstage.sourceforge.net/gazebo/xmlschema/#controller"
-       xmlns:interface="http://playerstage.sourceforge.net/gazebo/xmlschema/#interface"
-       xmlns:xacro="http://ros.org/wiki/xacro">
-	<xacro:macro name="ur5_arm_transmission" params="name">
-		<transmission name="shoulder_pan_trans" type="pr2_mechanism_model/SimpleTransmission">
-			<actuator name="shoulder_pan_motor"/>
-			<joint name="${name}shoulder_pan_joint"/>
-			<mechanicalReduction>1</mechanicalReduction>
+<robot xmlns:xacro="http://www.ros.org/wiki/xacro">
+	<xacro:macro name="ur5_arm_transmission" params="prefix">
+		<transmission name="${prefix}shoulder_pan_trans">
+			<type>transmission_interface/SimpleTransmission</type>
+			<joint name="${prefix}shoulder_pan_joint"/>
+			<actuator name="${prefix}shoulder_pan_motor">
+				<hardwareInterface>EffortJointInterface</hardwareInterface>
+				<mechanicalReduction>1</mechanicalReduction>
+			</actuator>
 		</transmission>
-		<transmission name="shoulder_lift_trans" type="pr2_mechanism_model/SimpleTransmission">
-			<actuator name="shoulder_lift_motor"/>
-			<joint name="${name}shoulder_lift_joint"/>
-			<mechanicalReduction>1</mechanicalReduction>
+		<transmission name="${prefix}shoulder_lift_trans">
+			<type>transmission_interface/SimpleTransmission</type>
+			<joint name="${prefix}shoulder_lift_joint"/>
+			<actuator name="${prefix}shoulder_lift_motor">
+				<hardwareInterface>EffortJointInterface</hardwareInterface>
+				<mechanicalReduction>1</mechanicalReduction>
+			</actuator>
 		</transmission>
-		<transmission name="elbow_trans" type="pr2_mechanism_model/SimpleTransmission">
-			<actuator name="elbow_motor"/>
-			<joint name="${name}elbow_joint"/>
-			<mechanicalReduction>1</mechanicalReduction>
+		<transmission name="${prefix}elbow_trans">
+			<type>transmission_interface/SimpleTransmission</type>
+			<joint name="${prefix}elbow_joint"/>
+			<actuator name="${prefix}elbow_motor">
+				<hardwareInterface>EffortJointInterface</hardwareInterface>
+				<mechanicalReduction>1</mechanicalReduction>
+			</actuator>
 		</transmission>
-		<transmission name="wrist_1_trans" type="pr2_mechanism_model/SimpleTransmission">
-			<actuator name="wrist_1_motor"/>
-			<joint name="${name}wrist_1_joint"/>
-			<mechanicalReduction>1</mechanicalReduction>
+		<transmission name="${prefix}wrist_1_trans">
+			<type>transmission_interface/SimpleTransmission</type>
+			<joint name="${prefix}wrist_1_joint"/>
+			<actuator name="${prefix}wrist_1_motor">
+				<hardwareInterface>EffortJointInterface</hardwareInterface>
+				<mechanicalReduction>1</mechanicalReduction>
+			</actuator>
 		</transmission>
-		<transmission name="wrist_2_trans" type="pr2_mechanism_model/SimpleTransmission">
-			<actuator name="wrist_2_motor"/>
-			<joint name="${name}wrist_2_joint"/>
-			<mechanicalReduction>1</mechanicalReduction>
+		<transmission name="${prefix}wrist_2_trans">
+			<type>transmission_interface/SimpleTransmission</type>
+			<joint name="${prefix}wrist_2_joint"/>
+			<actuator name="${prefix}wrist_2_motor">
+				<hardwareInterface>EffortJointInterface</hardwareInterface>
+				<mechanicalReduction>1</mechanicalReduction>
+			</actuator>
 		</transmission>
-		<transmission name="wrist_3_trans" type="pr2_mechanism_model/SimpleTransmission">
-			<actuator name="wrist_3_motor"/>
-			<joint name="${name}wrist_3_joint"/>
-			<mechanicalReduction>1</mechanicalReduction>
+		<transmission name="${prefix}wrist_3_trans">
+			<type>transmission_interface/SimpleTransmission</type>
+			<joint name="${prefix}wrist_3_joint"/>
+			<actuator name="${prefix}wrist_3_motor">
+				<hardwareInterface>EffortJointInterface</hardwareInterface>
+				<mechanicalReduction>1</mechanicalReduction>
+			</actuator>
 		</transmission>
 	</xacro:macro>

File: ur_description/urdf/ur5.urdf.xacro (robot description, xacro)
@@ -1,7 +1,4 @@
 <?xml version="1.0"?>
-<robot xmlns:sensor="http://playerstage.sourceforge.net/gazebo/xmlschema/#sensor"
-       xmlns:controller="http://playerstage.sourceforge.net/gazebo/xmlschema/#controller"
-       xmlns:interface="http://playerstage.sourceforge.net/gazebo/xmlschema/#interface"
-       xmlns:xacro="http://ros.org/wiki/xacro">
+<robot xmlns:xacro="http://www.ros.org/wiki/xacro">
   <xacro:include filename="$(find ur_description)/urdf/ur5.transmission.xacro" />
   <xacro:include filename="$(find ur_description)/urdf/ur5.gazebo.xacro" />
@@ -229,8 +226,6 @@
   </joint>
   <link name="${prefix}ee_link" />
-  <xacro:ur5_arm_transmission name="${prefix}" />
-  <gazebo reference="universal_robot">
-    <material>Gazebo/Blue</material>
-  </gazebo>
-</xacro:macro>
+  <xacro:ur5_arm_transmission prefix="${prefix}" />
+  <xacro:ur5_arm_gazebo prefix="${prefix}" />
+  </xacro:macro>
 </robot>

File: ur_description/urdf/ur5_joint_limited_robot.urdf (robot description, URDF)
Before this commit: robot ur5, 8 links, 7 joints
Joints:
- joint elbow_joint: limit lower=-3.14159265 upper=3.14159265 effort=10.0 velocity=3.14159265 -> lower=-3.14159265 upper=3.14159265 effort=150.0 velocity=3.14159265
- joint shoulder_lift_joint: limit lower=-3.14159265 upper=3.14159265 effort=10.0 velocity=3.14159265 -> lower=-3.14159265 upper=3.14159265 effort=150.0 velocity=3.14159265
- joint shoulder_pan_joint: limit lower=-3.14159265 upper=3.14159265 effort=10.0 velocity=3.14159265 -> lower=-3.14159265 upper=3.14159265 effort=150.0 velocity=3.14159265
- joint wrist_1_joint: limit lower=-3.14159265 upper=0.7853981625 effort=10.0 velocity=3.14159265 -> lower=-3.14159265 upper=0.7853981625 effort=28.0 velocity=3.14159265
- joint wrist_2_joint: limit lower=-3.14159265 upper=3.14159265 effort=10.0 velocity=3.14159265 -> lower=-3.14159265 upper=3.14159265 effort=28.0 velocity=3.14159265
- joint wrist_3_joint: limit lower=-3.14159265 upper=3.14159265 effort=10.0 velocity=3.14159265 -> lower=-3.14159265 upper=3.14159265 effort=28.0 velocity=3.14159265

File: ur_description/urdf/ur5_robot.urdf (robot description, URDF)
Before this commit: robot ur5, 8 links, 7 joints
Joints:
- joint elbow_joint: limit lower=-6.2831853 upper=6.2831853 effort=10.0 velocity=3.14159265 -> lower=-6.2831853 upper=6.2831853 effort=150.0 velocity=3.14159265
- joint shoulder_lift_joint: limit lower=-6.2831853 upper=6.2831853 effort=10.0 velocity=3.14159265 -> lower=-6.2831853 upper=6.2831853 effort=150.0 velocity=3.14159265
- joint shoulder_pan_joint: limit lower=-6.2831853 upper=6.2831853 effort=10.0 velocity=3.14159265 -> lower=-6.2831853 upper=6.2831853 effort=150.0 velocity=3.14159265
- joint wrist_1_joint: limit lower=-3.14159265 upper=0.7853981625 effort=10.0 velocity=3.14159265 -> lower=-3.14159265 upper=0.7853981625 effort=28.0 velocity=3.14159265
- joint wrist_2_joint: limit lower=-3.14159265 upper=3.14159265 effort=10.0 velocity=3.14159265 -> lower=-3.14159265 upper=3.14159265 effort=28.0 velocity=3.14159265
- joint wrist_3_joint: limit lower=-3.14159265 upper=3.14159265 effort=10.0 velocity=3.14159265 -> lower=-3.14159265 upper=3.14159265 effort=28.0 velocity=3.14159265

File: ur_description/urdf/ur5_robot.urdf.xacro (robot description, xacro)
@@ -1,7 +1,4 @@
 <?xml version="1.0"?>
-<robot xmlns:sensor="http://playerstage.sourceforge.net/gazebo/xmlschema/#sensor"
-       xmlns:controller="http://playerstage.sourceforge.net/gazebo/xmlschema/#controller"
-       xmlns:interface="http://playerstage.sourceforge.net/gazebo/xmlschema/#interface"
-       xmlns:xacro="http://playerstage.sourceforge.net/gazebo/xmlschema/#interface"
+<robot xmlns:xacro="http://www.ros.org/wiki/xacro"
        name="ur5" >
   <!-- common stuff -->
