Commit message: Imported upstream version '1.0.5' of 'upstream'

File: ur_description/urdf/ur10.transmission.xacro (robot description, xacro)
@@ -4,8 +4,7 @@
     <transmission name="${prefix}shoulder_pan_trans">
       <type>transmission_interface/SimpleTransmission</type>
-      <joint name="${prefix}shoulder_pan_joint">
+      <joint name="${prefix}shoulder_pan_joint"/>
+      <actuator name="${prefix}shoulder_pan_motor">
         <hardwareInterface>EffortJointInterface</hardwareInterface>
-      </joint>
-      <actuator name="${prefix}shoulder_pan_motor">
         <mechanicalReduction>1</mechanicalReduction>
       </actuator>
@@ -13,8 +12,7 @@
     <transmission name="${prefix}shoulder_lift_trans">
       <type>transmission_interface/SimpleTransmission</type>
-      <joint name="${prefix}shoulder_lift_joint">
+      <joint name="${prefix}shoulder_lift_joint"/>
+      <actuator name="${prefix}shoulder_lift_motor">
         <hardwareInterface>EffortJointInterface</hardwareInterface>
-      </joint>
-      <actuator name="${prefix}shoulder_lift_motor">
         <mechanicalReduction>1</mechanicalReduction>
       </actuator>
@@ -22,8 +20,7 @@
     <transmission name="${prefix}elbow_trans">
       <type>transmission_interface/SimpleTransmission</type>
-      <joint name="${prefix}elbow_joint">
+      <joint name="${prefix}elbow_joint"/>
+      <actuator name="${prefix}elbow_motor">
         <hardwareInterface>EffortJointInterface</hardwareInterface>
-      </joint>
-      <actuator name="${prefix}elbow_motor">
         <mechanicalReduction>1</mechanicalReduction>
       </actuator>
@@ -31,8 +28,7 @@
     <transmission name="${prefix}wrist_1_trans">
       <type>transmission_interface/SimpleTransmission</type>
-      <joint name="${prefix}wrist_1_joint">
+      <joint name="${prefix}wrist_1_joint"/>
+      <actuator name="${prefix}wrist_1_motor">
         <hardwareInterface>EffortJointInterface</hardwareInterface>
-      </joint>
-      <actuator name="${prefix}wrist_1_motor">
         <mechanicalReduction>1</mechanicalReduction>
       </actuator>
@@ -40,8 +36,7 @@
     <transmission name="${prefix}wrist_2_trans">
       <type>transmission_interface/SimpleTransmission</type>
-      <joint name="${prefix}wrist_2_joint">
+      <joint name="${prefix}wrist_2_joint"/>
+      <actuator name="${prefix}wrist_2_motor">
         <hardwareInterface>EffortJointInterface</hardwareInterface>
-      </joint>
-      <actuator name="${prefix}wrist_2_motor">
         <mechanicalReduction>1</mechanicalReduction>
       </actuator>
@@ -49,8 +44,7 @@
     <transmission name="${prefix}wrist_3_trans">
       <type>transmission_interface/SimpleTransmission</type>
-      <joint name="${prefix}wrist_3_joint">
+      <joint name="${prefix}wrist_3_joint"/>
+      <actuator name="${prefix}wrist_3_motor">
         <hardwareInterface>EffortJointInterface</hardwareInterface>
-      </joint>
-      <actuator name="${prefix}wrist_3_motor">
         <mechanicalReduction>1</mechanicalReduction>
       </actuator>

File: ur_description/urdf/ur5.transmission.xacro (robot description, xacro)
@@ -4,8 +4,7 @@
     <transmission name="${prefix}shoulder_pan_trans">
       <type>transmission_interface/SimpleTransmission</type>
-      <joint name="${prefix}shoulder_pan_joint">
+      <joint name="${prefix}shoulder_pan_joint"/>
+      <actuator name="${prefix}shoulder_pan_motor">
         <hardwareInterface>EffortJointInterface</hardwareInterface>
-      </joint>
-      <actuator name="${prefix}shoulder_pan_motor">
         <mechanicalReduction>1</mechanicalReduction>
       </actuator>
@@ -13,8 +12,7 @@
     <transmission name="${prefix}shoulder_lift_trans">
       <type>transmission_interface/SimpleTransmission</type>
-      <joint name="${prefix}shoulder_lift_joint">
+      <joint name="${prefix}shoulder_lift_joint"/>
+      <actuator name="${prefix}shoulder_lift_motor">
         <hardwareInterface>EffortJointInterface</hardwareInterface>
-      </joint>
-      <actuator name="${prefix}shoulder_lift_motor">
         <mechanicalReduction>1</mechanicalReduction>
       </actuator>
@@ -22,8 +20,7 @@
     <transmission name="${prefix}elbow_trans">
       <type>transmission_interface/SimpleTransmission</type>
-      <joint name="${prefix}elbow_joint">
+      <joint name="${prefix}elbow_joint"/>
+      <actuator name="${prefix}elbow_motor">
         <hardwareInterface>EffortJointInterface</hardwareInterface>
-      </joint>
-      <actuator name="${prefix}elbow_motor">
         <mechanicalReduction>1</mechanicalReduction>
       </actuator>
@@ -31,8 +28,7 @@
     <transmission name="${prefix}wrist_1_trans">
       <type>transmission_interface/SimpleTransmission</type>
-      <joint name="${prefix}wrist_1_joint">
+      <joint name="${prefix}wrist_1_joint"/>
+      <actuator name="${prefix}wrist_1_motor">
         <hardwareInterface>EffortJointInterface</hardwareInterface>
-      </joint>
-      <actuator name="${prefix}wrist_1_motor">
         <mechanicalReduction>1</mechanicalReduction>
       </actuator>
@@ -40,8 +36,7 @@
     <transmission name="${prefix}wrist_2_trans">
       <type>transmission_interface/SimpleTransmission</type>
-      <joint name="${prefix}wrist_2_joint">
+      <joint name="${prefix}wrist_2_joint"/>
+      <actuator name="${prefix}wrist_2_motor">
         <hardwareInterface>EffortJointInterface</hardwareInterface>
-      </joint>
-      <actuator name="${prefix}wrist_2_motor">
         <mechanicalReduction>1</mechanicalReduction>
       </actuator>
@@ -49,8 +44,7 @@
     <transmission name="${prefix}wrist_3_trans">
       <type>transmission_interface/SimpleTransmission</type>
-      <joint name="${prefix}wrist_3_joint">
+      <joint name="${prefix}wrist_3_joint"/>
+      <actuator name="${prefix}wrist_3_motor">
         <hardwareInterface>EffortJointInterface</hardwareInterface>
-      </joint>
-      <actuator name="${prefix}wrist_3_motor">
         <mechanicalReduction>1</mechanicalReduction>
       </actuator>

Commit message: Imported upstream version '1.1.5' of 'upstream'

File: ur_description/urdf/ur10.transmission.xacro (robot description, xacro)
@@ -4,7 +4,8 @@
     <transmission name="${prefix}shoulder_pan_trans">
       <type>transmission_interface/SimpleTransmission</type>
-      <joint name="${prefix}shoulder_pan_joint"/>
+      <joint name="${prefix}shoulder_pan_joint">
+        <hardwareInterface>EffortJointInterface</hardwareInterface>
+      </joint>
       <actuator name="${prefix}shoulder_pan_motor">
-        <hardwareInterface>EffortJointInterface</hardwareInterface>
         <mechanicalReduction>1</mechanicalReduction>
       </actuator>
@@ -12,7 +13,8 @@
     <transmission name="${prefix}shoulder_lift_trans">
       <type>transmission_interface/SimpleTransmission</type>
-      <joint name="${prefix}shoulder_lift_joint"/>
+      <joint name="${prefix}shoulder_lift_joint">
+        <hardwareInterface>EffortJointInterface</hardwareInterface>
+      </joint>
       <actuator name="${prefix}shoulder_lift_motor">
-        <hardwareInterface>EffortJointInterface</hardwareInterface>
         <mechanicalReduction>1</mechanicalReduction>
       </actuator>
@@ -20,7 +22,8 @@
     <transmission name="${prefix}elbow_trans">
       <type>transmission_interface/SimpleTransmission</type>
-      <joint name="${prefix}elbow_joint"/>
+      <joint name="${prefix}elbow_joint">
+        <hardwareInterface>EffortJointInterface</hardwareInterface>
+      </joint>
       <actuator name="${prefix}elbow_motor">
-        <hardwareInterface>EffortJointInterface</hardwareInterface>
         <mechanicalReduction>1</mechanicalReduction>
       </actuator>
@@ -28,7 +31,8 @@
     <transmission name="${prefix}wrist_1_trans">
       <type>transmission_interface/SimpleTransmission</type>
-      <joint name="${prefix}wrist_1_joint"/>
+      <joint name="${prefix}wrist_1_joint">
+        <hardwareInterface>EffortJointInterface</hardwareInterface>
+      </joint>
       <actuator name="${prefix}wrist_1_motor">
-        <hardwareInterface>EffortJointInterface</hardwareInterface>
         <mechanicalReduction>1</mechanicalReduction>
       </actuator>
@@ -36,7 +40,8 @@
     <transmission name="${prefix}wrist_2_trans">
       <type>transmission_interface/SimpleTransmission</type>
-      <joint name="${prefix}wrist_2_joint"/>
+      <joint name="${prefix}wrist_2_joint">
+        <hardwareInterface>EffortJointInterface</hardwareInterface>
+      </joint>
       <actuator name="${prefix}wrist_2_motor">
-        <hardwareInterface>EffortJointInterface</hardwareInterface>
         <mechanicalReduction>1</mechanicalReduction>
       </actuator>
@@ -44,7 +49,8 @@
     <transmission name="${prefix}wrist_3_trans">
       <type>transmission_interface/SimpleTransmission</type>
-      <joint name="${prefix}wrist_3_joint"/>
+      <joint name="${prefix}wrist_3_joint">
+        <hardwareInterface>EffortJointInterface</hardwareInterface>
+      </joint>
       <actuator name="${prefix}wrist_3_motor">
-        <hardwareInterface>EffortJointInterface</hardwareInterface>
         <mechanicalReduction>1</mechanicalReduction>
       </actuator>

File: ur_description/urdf/ur5.transmission.xacro (robot description, xacro)
@@ -4,7 +4,8 @@
     <transmission name="${prefix}shoulder_pan_trans">
       <type>transmission_interface/SimpleTransmission</type>
-      <joint name="${prefix}shoulder_pan_joint"/>
+      <joint name="${prefix}shoulder_pan_joint">
+        <hardwareInterface>EffortJointInterface</hardwareInterface>
+      </joint>
       <actuator name="${prefix}shoulder_pan_motor">
-        <hardwareInterface>EffortJointInterface</hardwareInterface>
         <mechanicalReduction>1</mechanicalReduction>
       </actuator>
@@ -12,7 +13,8 @@
     <transmission name="${prefix}shoulder_lift_trans">
       <type>transmission_interface/SimpleTransmission</type>
-      <joint name="${prefix}shoulder_lift_joint"/>
+      <joint name="${prefix}shoulder_lift_joint">
+        <hardwareInterface>EffortJointInterface</hardwareInterface>
+      </joint>
       <actuator name="${prefix}shoulder_lift_motor">
-        <hardwareInterface>EffortJointInterface</hardwareInterface>
         <mechanicalReduction>1</mechanicalReduction>
       </actuator>
@@ -20,7 +22,8 @@
     <transmission name="${prefix}elbow_trans">
       <type>transmission_interface/SimpleTransmission</type>
-      <joint name="${prefix}elbow_joint"/>
+      <joint name="${prefix}elbow_joint">
+        <hardwareInterface>EffortJointInterface</hardwareInterface>
+      </joint>
       <actuator name="${prefix}elbow_motor">
-        <hardwareInterface>EffortJointInterface</hardwareInterface>
         <mechanicalReduction>1</mechanicalReduction>
       </actuator>
@@ -28,7 +31,8 @@
     <transmission name="${prefix}wrist_1_trans">
       <type>transmission_interface/SimpleTransmission</type>
-      <joint name="${prefix}wrist_1_joint"/>
+      <joint name="${prefix}wrist_1_joint">
+        <hardwareInterface>EffortJointInterface</hardwareInterface>
+      </joint>
       <actuator name="${prefix}wrist_1_motor">
-        <hardwareInterface>EffortJointInterface</hardwareInterface>
         <mechanicalReduction>1</mechanicalReduction>
       </actuator>
@@ -36,7 +40,8 @@
     <transmission name="${prefix}wrist_2_trans">
       <type>transmission_interface/SimpleTransmission</type>
-      <joint name="${prefix}wrist_2_joint"/>
+      <joint name="${prefix}wrist_2_joint">
+        <hardwareInterface>EffortJointInterface</hardwareInterface>
+      </joint>
       <actuator name="${prefix}wrist_2_motor">
-        <hardwareInterface>EffortJointInterface</hardwareInterface>
         <mechanicalReduction>1</mechanicalReduction>
       </actuator>
@@ -44,7 +49,8 @@
     <transmission name="${prefix}wrist_3_trans">
       <type>transmission_interface/SimpleTransmission</type>
-      <joint name="${prefix}wrist_3_joint"/>
+      <joint name="${prefix}wrist_3_joint">
+        <hardwareInterface>EffortJointInterface</hardwareInterface>
+      </joint>
       <actuator name="${prefix}wrist_3_motor">
-        <hardwareInterface>EffortJointInterface</hardwareInterface>
         <mechanicalReduction>1</mechanicalReduction>
       </actuator>
