Commit message: Rebase from 'release/hydro/ur_description'

File: urdf/ur10_joint_limited.urdf.xacro (robot description, xacro)
@@ -64,5 +64,5 @@
     <origin xyz="0.0 0.0 ${shoulder_height}" rpy="0.0 0.0 0.0" />
     <axis xyz="0.0 0.0 1.0" />
-    <limit lower="${-2.0 * pi}" upper="${2.0 * pi}" effort="330.0" velocity="2.16"/>
+    <limit lower="${-pi}" upper="${pi}" effort="330.0" velocity="2.16"/>
     <dynamics damping="1.2" friction="0.0"/>
   </joint>
@@ -90,5 +90,5 @@
     <origin xyz="0.0 ${shoulder_offset} 0.0" rpy="0.0 ${pi / 2.0} 0.0" />
     <axis xyz="0.0 1.0 0.0" />
-    <limit lower="${-2.0 * pi}" upper="${2.0 * pi}" effort="10.0" velocity="${pi}"/>
+    <limit lower="${-pi}" upper="${pi}" effort="10.0" velocity="${pi}"/>
     <dynamics damping="1.2" friction="0.0"/>
   </joint>
@@ -118,5 +118,5 @@
     <origin xyz="0.0 ${-elbow_offset} ${upper_arm_length}" rpy="0.0 0.0 0.0" />
     <axis xyz="0.0 1.0 0.0" />
-    <limit lower="${-2.0 * pi}" upper="${2.0 * pi}" effort="150.0" velocity="${pi}"/>
+    <limit lower="${-pi}" upper="${pi}" effort="150.0" velocity="${pi}"/>
     <dynamics damping="0.6" friction="0.0"/>
   </joint>
@@ -144,5 +144,5 @@
     <origin xyz="0.0 0.0 ${forearm_length}" rpy="0.0 ${pi / 2.0} 0.0" />
     <axis xyz="0.0 1.0 0.0" />
-    <limit lower="${-2.0 * pi}" upper="${2.0 * pi}" effort="54.0" velocity="${pi}"/>
+    <limit lower="${-pi}" upper="${pi}" effort="54.0" velocity="${pi}"/>
     <dynamics damping="0.6" friction="0.0"/>
   </joint>
@@ -172,5 +172,5 @@
     <origin xyz="0.0 ${wrist_1_length} 0.0" rpy="0.0 0.0 0.0" />
     <axis xyz="0.0 0.0 1.0" />
-    <limit lower="${-2.0 * pi}" upper="${2.0 * pi}" effort="54.0" velocity="${pi}"/>
+    <limit lower="${-pi}" upper="${pi}" effort="54.0" velocity="${pi}"/>
     <dynamics damping="0.6" friction="0.0"/>
   </joint>
@@ -200,5 +200,5 @@
     <origin xyz="0.0 0.0 ${wrist_2_length}" rpy="0.0 0.0 0.0" />
     <axis xyz="0.0 1.0 0.0" />
-    <limit lower="${-2.0 * pi}" upper="${2.0 * pi}" effort="54.0" velocity="${pi}"/>
+    <limit lower="${-pi}" upper="${pi}" effort="54.0" velocity="${pi}"/>
     <dynamics damping="0.6" friction="0.0"/>
   </joint>

File: urdf/ur10_joint_limited_robot.urdf (robot description, URDF)
Before this commit: robot ur5, 8 links, 7 joints
Links:
- link base_link: geometry collision mesh filename=package://ur_description/meshes/ur10/collision/Base.stl; visual mesh filename=package://ur_description/meshes/ur10/visual/Base.stl
- link forearm_link: geometry collision mesh filename=package://ur_description/meshes/ur10/collision/Forearm.stl; visual mesh filename=package://ur_description/meshes/ur10/visual/Forearm.stl
- link shoulder_link: geometry collision mesh filename=package://ur_description/meshes/ur10/collision/Shoulder.stl; visual mesh filename=package://ur_description/meshes/ur10/visual/Shoulder.stl
- link upper_arm_link: geometry collision mesh filename=package://ur_description/meshes/ur10/collision/UpperArm.stl; visual mesh filename=package://ur_description/meshes/ur10/visual/UpperArm.stl
- link wrist_1_link: geometry collision mesh filename=package://ur_description/meshes/ur10/collision/Wrist1.stl; visual mesh filename=package://ur_description/meshes/ur10/visual/Wrist1.stl
- link wrist_2_link: geometry collision mesh filename=package://ur_description/meshes/ur10/collision/Wrist2.stl; visual mesh filename=package://ur_description/meshes/ur10/visual/Wrist2.stl
- link wrist_3_link: geometry collision mesh filename=package://ur_description/meshes/ur10/collision/Wrist3.stl; visual mesh filename=package://ur_description/meshes/ur10/visual/Wrist3.stl
Joints:
- joint ee_fixed_joint: origin xyz=0.0 0.0823 0.0 rpy=0.0 0.0 1.570796325 -> xyz=0.0 0.0857 0.0 rpy=0.0 0.0 1.570796325
- joint elbow_joint: axis 0 1 0 -> 0.0 1.0 0.0; origin xyz=0.0 -0.1197 0.425 rpy=0.0 0.0 0.0 -> xyz=0.0 -0.12817 0.60186 rpy=0.0 0.0 0.0
- joint shoulder_lift_joint: axis 0 1 0 -> 0.0 1.0 0.0; limit lower=-3.14159265 upper=3.14159265 effort=150.0 velocity=3.14159265 -> lower=-3.14159265 upper=3.14159265 effort=10.0 velocity=3.14159265; origin xyz=0.0 0.13585 0.0 rpy=0.0 1.570796325 0.0 -> xyz=0.0 0.1704 0.0 rpy=0.0 1.570796325 0.0
- joint shoulder_pan_joint: axis 0 0 1 -> 0.0 0.0 1.0; limit lower=-3.14159265 upper=3.14159265 effort=150.0 velocity=3.14159265 -> lower=-3.14159265 upper=3.14159265 effort=330.0 velocity=2.16; origin xyz=0.0 0.0 0.089159 rpy=0.0 0.0 0.0 -> xyz=0.0 0.0 0.128 rpy=0.0 0.0 0.0
- joint wrist_1_joint: axis 0 1 0 -> 0.0 1.0 0.0; limit lower=-3.14159265 upper=0.7853981625 effort=28.0 velocity=3.14159265 -> lower=-3.14159265 upper=3.14159265 effort=54.0 velocity=3.14159265; origin xyz=0.0 0.0 0.39225 rpy=0.0 1.570796325 0.0 -> xyz=0.0 0.0 0.56415 rpy=0.0 1.570796325 0.0
- joint wrist_2_joint: axis 0 0 1 -> 0.0 0.0 1.0; limit lower=-3.14159265 upper=3.14159265 effort=28.0 velocity=3.14159265 -> lower=-3.14159265 upper=3.14159265 effort=54.0 velocity=3.14159265; origin xyz=0.0 0.093 0.0 rpy=0.0 0.0 0.0 -> xyz=0.0 0.11279 0.0 rpy=0.0 0.0 0.0
- joint wrist_3_joint: axis 0 1 0 -> 0.0 1.0 0.0; limit lower=-3.14159265 upper=3.14159265 effort=28.0 velocity=3.14159265 -> lower=-3.14159265 upper=3.14159265 effort=54.0 velocity=3.14159265; origin xyz=0.0 0.0 0.09465 rpy=0.0 0.0 0.0 -> xyz=0.0 0.0 0.11279 rpy=0.0 0.0 0.0

File: urdf/ur10_joint_limited_robot.urdf.xacro (robot description, xacro)
@@ -1,11 +1,11 @@
 <?xml version="1.0"?>
 <robot xmlns:xacro="http://www.ros.org/wiki/xacro"
-       name="ur5" >
+       name="ur10" >
   <!-- common stuff -->
   <xacro:include filename="$(find ur_description)/urdf/gazebo.urdf.xacro" />
-  <!-- ur5 -->
-  <xacro:include filename="$(find ur_description)/urdf/ur5.urdf.xacro" />
+  <!-- ur10 -->
+  <xacro:include filename="$(find ur_description)/urdf/ur10_joint_limited.urdf.xacro" />
   <!-- arm -->
-  <xacro:ur5_robot prefix="">
-  </xacro:ur5_robot>
+  <xacro:ur10_robot prefix="">
+  </xacro:ur10_robot>
 </robot>

File: urdf/ur10_robot.urdf (robot description, URDF)
Before this commit: robot ur5, 8 links, 7 joints
Links:
- link base_link: geometry collision mesh filename=package://ur_description/meshes/ur10/collision/Base.stl; visual mesh filename=package://ur_description/meshes/ur10/visual/Base.stl
- link forearm_link: geometry collision mesh filename=package://ur_description/meshes/ur10/collision/Forearm.stl; visual mesh filename=package://ur_description/meshes/ur10/visual/Forearm.stl
- link shoulder_link: geometry collision mesh filename=package://ur_description/meshes/ur10/collision/Shoulder.stl; visual mesh filename=package://ur_description/meshes/ur10/visual/Shoulder.stl
- link upper_arm_link: geometry collision mesh filename=package://ur_description/meshes/ur10/collision/UpperArm.stl; visual mesh filename=package://ur_description/meshes/ur10/visual/UpperArm.stl
- link wrist_1_link: geometry collision mesh filename=package://ur_description/meshes/ur10/collision/Wrist1.stl; visual mesh filename=package://ur_description/meshes/ur10/visual/Wrist1.stl
- link wrist_2_link: geometry collision mesh filename=package://ur_description/meshes/ur10/collision/Wrist2.stl; visual mesh filename=package://ur_description/meshes/ur10/visual/Wrist2.stl
- link wrist_3_link: geometry collision mesh filename=package://ur_description/meshes/ur10/collision/Wrist3.stl; visual mesh filename=package://ur_description/meshes/ur10/visual/Wrist3.stl
Joints:
- joint ee_fixed_joint: origin xyz=0.0 0.0823 0.0 rpy=0.0 0.0 1.570796325 -> xyz=0.0 0.0857 0.0 rpy=0.0 0.0 1.570796325
- joint elbow_joint: axis 0 1 0 -> 0.0 1.0 0.0; limit lower=-3.14159265 upper=3.14159265 effort=150.0 velocity=3.14159265 -> lower=-6.2831853 upper=6.2831853 effort=150.0 velocity=3.14159265; origin xyz=0.0 -0.1197 0.425 rpy=0.0 0.0 0.0 -> xyz=0.0 -0.12817 0.60186 rpy=0.0 0.0 0.0
- joint shoulder_lift_joint: axis 0 1 0 -> 0.0 1.0 0.0; limit lower=-3.14159265 upper=3.14159265 effort=150.0 velocity=3.14159265 -> lower=-6.2831853 upper=6.2831853 effort=10.0 velocity=3.14159265; origin xyz=0.0 0.13585 0.0 rpy=0.0 1.570796325 0.0 -> xyz=0.0 0.1704 0.0 rpy=0.0 1.570796325 0.0
- joint shoulder_pan_joint: axis 0 0 1 -> 0.0 0.0 1.0; limit lower=-3.14159265 upper=3.14159265 effort=150.0 velocity=3.14159265 -> lower=-6.2831853 upper=6.2831853 effort=330.0 velocity=2.16; origin xyz=0.0 0.0 0.089159 rpy=0.0 0.0 0.0 -> xyz=0.0 0.0 0.128 rpy=0.0 0.0 0.0
- joint wrist_1_joint: axis 0 1 0 -> 0.0 1.0 0.0; limit lower=-3.14159265 upper=0.7853981625 effort=28.0 velocity=3.14159265 -> lower=-6.2831853 upper=6.2831853 effort=54.0 velocity=3.14159265; origin xyz=0.0 0.0 0.39225 rpy=0.0 1.570796325 0.0 -> xyz=0.0 0.0 0.56415 rpy=0.0 1.570796325 0.0
- joint wrist_2_joint: axis 0 0 1 -> 0.0 0.0 1.0; limit lower=-3.14159265 upper=3.14159265 effort=28.0 velocity=3.14159265 -> lower=-6.2831853 upper=6.2831853 effort=54.0 velocity=3.14159265; origin xyz=0.0 0.093 0.0 rpy=0.0 0.0 0.0 -> xyz=0.0 0.11279 0.0 rpy=0.0 0.0 0.0
- joint wrist_3_joint: axis 0 1 0 -> 0.0 1.0 0.0; limit lower=-3.14159265 upper=3.14159265 effort=28.0 velocity=3.14159265 -> lower=-6.2831853 upper=6.2831853 effort=54.0 velocity=3.14159265; origin xyz=0.0 0.0 0.09465 rpy=0.0 0.0 0.0 -> xyz=0.0 0.0 0.11279 rpy=0.0 0.0 0.0

File: urdf/ur5_joint_limited.urdf.xacro (robot description, xacro)
@@ -67,5 +67,5 @@
     <origin xyz="0.0 0.0 ${shoulder_height}" rpy="0.0 0.0 0.0" />
     <axis xyz="0 0 1" />
-    <limit lower="${-2.0 * pi}" upper="${2.0 * pi}" effort="150.0" velocity="${pi}"/>
+    <limit lower="${-pi}" upper="${pi}" effort="150.0" velocity="${pi}"/>
     <dynamics damping="0.4" friction="0.0"/>
   </joint>
@@ -93,5 +93,5 @@
     <origin xyz="0.0 ${shoulder_offset} 0.0" rpy="0.0 ${pi / 2.0} 0.0" />
     <axis xyz="0 1 0" />
-    <limit lower="${-2.0 * pi}" upper="${2.0 * pi}" effort="150.0" velocity="${pi}"/>
+    <limit lower="${-pi}" upper="${pi}" effort="150.0" velocity="${pi}"/>
     <dynamics damping="0.4" friction="0.0"/>
   </joint>
@@ -120,5 +120,5 @@
     <origin xyz="0.0 ${-elbow_offset} ${upper_arm_length}" rpy="0.0 0.0 0.0" />
     <axis xyz="0 1 0" />
-    <limit lower="${-2.0 * pi}" upper="${2.0 * pi}" effort="150.0" velocity="${pi}"/>
+    <limit lower="${-pi}" upper="${pi}" effort="150.0" velocity="${pi}"/>
     <dynamics damping="0.4" friction="0.0"/>
   </joint>

File: urdf/ur5_joint_limited_robot.urdf.xacro (robot description, xacro)
@@ -5,5 +5,5 @@
   <xacro:include filename="$(find ur_description)/urdf/gazebo.urdf.xacro" />
   <!-- ur5 -->
-  <xacro:include filename="$(find ur_description)/urdf/ur5.urdf.xacro" />
+  <xacro:include filename="$(find ur_description)/urdf/ur5_joint_limited.urdf.xacro" />
   <!-- arm -->
   <xacro:ur5_robot prefix="">
